File: digits/digits.kicad_pcb (KiCad board)
At the start: 2 copper layers, 70 x 119 mm, 267 parts, among them J1 SOLDER, J2 EDGE_CONNECT, Q1 BSS84, Q10 BSS84, Q11 BSS84, Q12 BSS84, Q13 BSS84, Q14 BSS84, Q2 BSS84, Q3 BSS84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

Commit message: Added fiducials, fixed typo on the connector, added the correct origin, added a version number
Parts:
- added FID1: Fiducial, Fiducial:Fiducial_1mm_Mask3mm, F.Cu at (122.5, 139.0)
- added FID2: Fiducial, Fiducial:Fiducial_1mm_Mask3mm, F.Cu at (177.0, 133.5)
- added FID3: Fiducial, Fiducial:Fiducial_1mm_Mask3mm, F.Cu at (171.5, 30.0)
- added FID4: Fiducial, Fiducial:Fiducial_1mm_Mask3mm, F.Cu at (117.0, 35.5)
Other:
- board text added: "V1.1"

Commit message: didn't even need that part
Parts:
- removed U2: 74AHC244, Package_SO:TSSOP-20_4.4x5mm_P0.5mm
- added REF**: boykisser_5mm, digits:boykisser_5mm, F.Cu at (158.8, 90.5)
- moved R99 9.40 mm to (146.8, 102.1)
- moved C2 0.84 mm to (150.5, 91.0)
Connections:
- R99 pad 2: Net-(U2-2Y3) -> Net-(U1-QH)
- U1 pad 1: Net-(U1-QB) -> /B
- U1 pad 15: Net-(U1-QA) -> /A
- U1 pad 2: Net-(U1-QC) -> /C
- U1 pad 3: Net-(U1-QD) -> /D
- U1 pad 4: Net-(U1-QE) -> /E
- U1 pad 5: Net-(U1-QF) -> /F
- U1 pad 6: Net-(U1-QG) -> /G
Routing:
- net /B: track 76.9 -> 94.7 mm, vias 2 -> 4
- net Net-(U1-QA): track 17.5 -> 0.00 mm, vias 2 -> 0
- net Net-(U1-QB): track 17.2 -> 0.00 mm
- net Net-(U1-QC): track 16.9 -> 0.00 mm
- net Net-(U1-QD): track 16.6 -> 0.00 mm
- net /C: track 73.0 -> 89.4 mm, vias 2 -> 4
- net Net-(U1-QH): track 18.7 -> 2.38 mm, vias 3 -> 0
- net +5V: track 502.5 -> 487.2 mm
- net /A: track 73.6 -> 88.3 mm, vias 2 -> 6
- net Net-(U1-QE): track 13.4 -> 0.00 mm
- net Net-(U1-QF): track 13.2 -> 0.00 mm
- net Net-(U1-QG): track 12.5 -> 0.00 mm
- net /E: track 93.5 -> 81.7 mm
- net /F: track 101.5 -> 90.5 mm
- net /D: track 42.0 -> 35.0 mm, vias 3 -> 5
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